Commit message: 增加了realtime-servo

File: er7robot_arm_description/urdf/er7.xacro (robot description, xacro)
@@ -13,6 +13,4 @@
   </material>
   <xacro:macro name="estun_robot" params=" prefix parent_link attach_xyz attach_rpy">
-    <!-- ================== 可配置参数 ================== -->
-    <!-- ================== 宏定义 ================== -->
     <!-- 全局参数 -->
     <xacro:property name="pkg" value="er7robot_arm_description" />
@@ -187,5 +185,5 @@
                         upper="6.28319"/>
     <!-- ================== 控制接口 ================== -->
-    <ros2_control name="${prefix}er7_ros2_control" type="system">
+    <!-- <ros2_control name="${prefix}er7_ros2_control" type="system">
       <hardware>
         <plugin>gazebo_ros2_control/GazeboSystem</plugin>
@@ -269,5 +267,5 @@
         <state_interface name="effort"/>
       </joint>
-    </ros2_control>
+    </ros2_control> -->
   </xacro:macro>
 </robot>

File: er7robot_arm_description/urdf/er7_two_arm.xacro (robot description, xacro)
@@ -5,11 +5,11 @@
     <xacro:estun_robot prefix="laser_" parent_link="base_link" attach_xyz="1.0 0 0" attach_rpy="0 0 -1.57"/>
     <link name="base_link"/>
-    <gazebo>
-        <plugin filename="libgazebo_ros2_control.so" name="gazebo_ros2_control">
+    <!-- <gazebo>
+        <plugin filename="libgazebo_ros2_control.so" name="gazebo_ros2_control"> -->
             <!--launch controller manager to manage joint_state_boardcaster and my_arm_group_controller-->
-            <parameters>$(find er7robot_two_arm_moveit_config)/config/ros2_controllers.yaml</parameters>
+            <!-- <parameters>$(find er7robot_two_arm_moveit_config)/config/ros2_controllers.yaml</parameters>  -->
             <!--declare where to get robot_description-->
-            <robot_param_node>robot_state_publisher</robot_param_node>
+            <!-- <robot_param_node>robot_state_publisher</robot_param_node>
         </plugin>
-    </gazebo>
+    </gazebo> -->
 </robot>

File: er7robot_two_arm_moveit_config/config/er7robot.ros2_control.xacro (robot description, xacro)
@@ -2,5 +2,5 @@
 <robot xmlns:xacro="http://www.ros.org/wiki/xacro">
     <xacro:macro name="er7robot_ros2_control" params="name initial_positions_file">
-        <xacro:property name="initial_positions" value="${xacro.load_yaml(initial_positions_file)['initial_positions']}"/>
+        <xacro:property name="initial_positions" value="${load_yaml(initial_positions_file)['initial_positions']}"/>
         <ros2_control name="${name}" type="system">
             <hardware>
@@ -10,73 +10,97 @@
             <joint name="camera_joint_1">
                 <command_interface name="position"/>
+                <command_interface name="velocity"/>
                 <state_interface name="position">
                   <param name="initial_value">${initial_positions['camera_joint_1']}</param>
                 </state_interface>
+                <state_interface name="velocity"/>
             </joint>
             <joint name="camera_joint_2">
                 <command_interface name="position"/>
+                <command_interface name="velocity"/>
                 <state_interface name="position">
                   <param name="initial_value">${initial_positions['camera_joint_2']}</param>
                 </state_interface>
+                <state_interface name="velocity"/>
             </joint>
             <joint name="camera_joint_3">
                 <command_interface name="position"/>
+                <command_interface name="velocity"/>
                 <state_interface name="position">
                   <param name="initial_value">${initial_positions['camera_joint_3']}</param>
                 </state_interface>
+                <state_interface name="velocity"/>
             </joint>
             <joint name="camera_joint_4">
                 <command_interface name="position"/>
+                <command_interface name="velocity"/>
                 <state_interface name="position">
                   <param name="initial_value">${initial_positions['camera_joint_4']}</param>
                 </state_interface>
+                <state_interface name="velocity"/>
             </joint>
             <joint name="camera_joint_5">
                 <command_interface name="position"/>
+                <command_interface name="velocity"/>
                 <state_interface name="position">
                   <param name="initial_value">${initial_positions['camera_joint_5']}</param>
                 </state_interface>
+                <state_interface name="velocity"/>
             </joint>
             <joint name="camera_joint_6">
                 <command_interface name="position"/>
+                <command_interface name="velocity"/>
                 <state_interface name="position">
                   <param name="initial_value">${initial_positions['camera_joint_6']}</param>
                 </state_interface>
+                <state_interface name="velocity"/>
             </joint>
             <joint name="laser_joint_1">
                 <command_interface name="position"/>
+                <command_interface name="velocity"/>
                 <state_interface name="position">
                   <param name="initial_value">${initial_positions['laser_joint_1']}</param>
                 </state_interface>
+                <state_interface name="velocity"/>
             </joint>
             <joint name="laser_joint_2">
                 <command_interface name="position"/>
+                <command_interface name="velocity"/>
                 <state_interface name="position">
                   <param name="initial_value">${initial_positions['laser_joint_2']}</param>
                 </state_interface>
+                <state_interface name="velocity"/>
             </joint>
             <joint name="laser_joint_3">
                 <command_interface name="position"/>
+                <command_interface name="velocity"/>
                 <state_interface name="position">
                   <param name="initial_value">${initial_positions['laser_joint_3']}</param>
                 </state_interface>
+                <state_interface name="velocity"/>
             </joint>
             <joint name="laser_joint_4">
                 <command_interface name="position"/>
+                <command_interface name="velocity"/>
                 <state_interface name="position">
                   <param name="initial_value">${initial_positions['laser_joint_4']}</param>
                 </state_interface>
+                <state_interface name="velocity"/>
             </joint>
             <joint name="laser_joint_5">
                 <command_interface name="position"/>
+                <command_interface name="velocity"/>
                 <state_interface name="position">
                   <param name="initial_value">${initial_positions['laser_joint_5']}</param>
                 </state_interface>
+                <state_interface name="velocity"/>
             </joint>
             <joint name="laser_joint_6">
                 <command_interface name="position"/>
+                <command_interface name="velocity"/>
                 <state_interface name="position">
                   <param name="initial_value">${initial_positions['laser_joint_6']}</param>
                 </state_interface>
+                <state_interface name="velocity"/>
             </joint>
         </ros2_control>
